File: gwIthoRFT.kicad_pcb (KiCad board)
At the start: 2 copper layers, 54.6 x 18 mm, 2 parts, among them U1 ProMicro, U2 E07-900M10S

Commit message: gwIthoRFT v2.0.0
Parts:
- moved U1 0.39 mm to (141.0, 85.1)
Connections:
- U1 pad 13: /MISO -> /CSN
- U1 pad 15: /SCK -> /MISO
- U1 pad 16: /CSN -> /SCK
Routing:
- net /CSN: track 32.9 -> 26.1 mm
- net /MISO: track 22.7 -> 28.7 mm
- net /SCK: track 29.5 -> 32.8 mm
- net +3V3: track 33.8 -> 32.2 mm
- net /MOSI: track 26.0 -> 26.9 mm
- net GND: vias 0 -> 9
Other:
- board text added: "v2.0.0"
- board text removed: "v1.0.0"
