File: gwIthoRFT.kicad_sch (KiCad schematic)
At the start: 2 parts, among them U1 ProMicro, U2 E07-900M10S

Commit message: gwIthoRFT v2.0.0
Connections:
- net CSN: now also U1.13 (D10); no longer U1.16 (B1)
- net MISO: now also U1.15 (D14(MISO)); no longer U1.13 (B6)
- net SCK: now also U1.16 (D15(SCK)); no longer U1.15 (B3)
Changed lines of the file:
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@@
     (effects (font (size 1.27 1.27)) (justify right bottom))
   )
-  (label "MISO" (at 140.97 60.96 180) (fields_autoplaced)
+  (label "MISO" (at 140.97 55.88 180) (fields_autoplaced)
     (effects (font (size 1.27 1.27)) (justify right bottom))
   )
-  (label "SCK" (at 140.97 55.88 180) (fields_autoplaced)
+  (label "SCK" (at 140.97 53.34 180) (fields_autoplaced)
     (effects (font (size 1.27 1.27)) (justify right bottom))
   )
@@
     (effects (font (size 1.27 1.27)) (justify right bottom))
   )
-  (label "CSN" (at 140.97 53.34 180) (fields_autoplaced)
+  (label "CSN" (at 140.97 60.96 180) (fields_autoplaced)
     (effects (font (size 1.27 1.27)) (justify right bottom))
   )
